File: Eagle/opt_isp6_prg_header.brd (EAGLE design)
At the start: 35.6 x 17.8 mm, 5 parts, among them J1 AVR_SPI_PROG_3X2NS

Commit message: Update opt_isp6_prg_header.brd
Routing:
- net SCLK: track 56.6 -> 55.7 mm
Other:
- board text added: "GND"
- board text added: "MISO"
- board text added: "MOSI"
- board text added: "RST"
- board text added: "SCK"
- board text added: "VCC"

Commit message: Update opt_isp6_prg_header.brd
Other:
- outline, holes or cut-outs redrawn
Changed lines of the file:
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@@
 <board>
 <plain>
-<wire x1="0" y1="0" x2="35.611" y2="0" width="0" layer="20"/>
-<wire x1="35.611" y1="0" x2="35.611" y2="17.77" width="0" layer="20"/>
-<wire x1="35.611" y1="17.77" x2="0" y2="17.77" width="0" layer="20"/>
-<wire x1="0" y1="17.77" x2="0" y2="0" width="0" layer="20"/>
+<wire x1="1.27" y1="0" x2="34.29" y2="0" width="0.0762" layer="20"/>
+<wire x1="0" y1="16.51" x2="0" y2="1.27" width="0.0762" layer="20"/>
 <wire x1="9.525" y1="15.367" x2="15.875" y2="15.367" width="0.1524" layer="21"/>
 <wire x1="15.875" y1="15.367" x2="15.875" y2="2.413" width="0.1524" layer="21"/>
@@
 <wire x1="34.29" y1="6.35" x2="34.29" y2="11.43" width="0.1524" layer="21"/>
 <wire x1="34.29" y1="11.43" x2="35.56" y2="11.43" width="0.1524" layer="21"/>
+<wire x1="0" y1="16.51" x2="1.27" y2="17.78" width="0.0762" layer="20" curve="-90"/>
+<wire x1="34.29" y1="17.78" x2="35.56" y2="16.51" width="0.0762" layer="20" curve="-90"/>
+<wire x1="35.56" y1="1.27" x2="34.29" y2="0" width="0.0762" layer="20" curve="-90"/>
+<wire x1="1.27" y1="0" x2="0" y2="1.27" width="0.0762" layer="20" curve="-90"/>
+<wire x1="1.27" y1="17.78" x2="34.29" y2="17.78" width="0.0762" layer="20"/>
+<wire x1="35.56" y1="16.51" x2="35.56" y2="1.27" width="0.0762" layer="20"/>
 </plain>
 <attributes>
@@
 </polygon>
 <via x="17.78" y="7.62" extent="1-16" drill="0.35"/>
-<via x="27.94" y="11.43" extent="1-16" drill="0.35"/>
+<via x="27.813" y="11.43" extent="1-16" drill="0.35"/>
 <via x="32.385" y="15.875" extent="1-16" drill="0.35"/>
 <via x="32.385" y="1.905" extent="1-16" drill="0.35"/>
@@
 <wire x1="20.828" y1="3.048" x2="21.59" y2="3.81" width="0.4064" layer="16"/>
 <wire x1="34.035" y1="3.81" x2="29.21" y2="3.81" width="0.4064" layer="1"/>
-<wire x1="29.21" y1="3.81" x2="27.94" y2="2.54" width="0.4064" layer="1"/>
-<via x="27.94" y="2.54" extent="1-16" drill="0.35"/>
-<wire x1="27.94" y1="2.54" x2="27.432" y2="2.032" width="0.4064" layer="16"/>
+<wire x1="29.21" y1="3.81" x2="27.813" y2="2.413" width="0.4064" layer="1"/>
+<via x="27.813" y="2.413" extent="1-16" drill="0.35"/>
+<wire x1="27.813" y1="2.413" x2="27.432" y2="2.032" width="0.4064" layer="16"/>
 <wire x1="27.432" y1="2.032" x2="23.368" y2="2.032" width="0.4064" layer="16"/>
 <wire x1="23.368" y1="2.032" x2="21.59" y2="3.81" width="0.4064" layer="16"/>
@@
 <wire x1="11.43" y1="2.54" x2="2.54" y2="2.54" width="0.4064" layer="1"/>
 <wire x1="11.43" y1="6.35" x2="11.43" y2="2.54" width="0.4064" layer="1"/>
-<via x="27.305" y="8.89" extent="1-16" drill="0.35"/>
-<wire x1="27.305" y1="8.89" x2="34.035" y2="8.89" width="0.4064" layer="1"/>
+<via x="27.813" y="8.89" extent="1-16" drill="0.35"/>
+<wire x1="27.813" y1="8.89" x2="34.035" y2="8.89" width="0.4064" layer="1"/>
 <wire x1="11.43" y1="2.54" x2="17.75173125" y2="2.54" width="0.4064" layer="1"/>
 <wire x1="17.75173125" y1="2.54" x2="19.07253125" y2="1.2192" width="0.4064" layer="1"/>
 <wire x1="19.07253125" y1="1.2192" x2="25.2222" y2="1.2192" width="0.4064" layer="1"/>
-<via x="27.3332" y="4.445" extent="1-16" drill="0.35"/>
-<wire x1="25.2222" y1="1.2192" x2="27.3332" y2="3.3302" width="0.4064" layer="1"/>
-<wire x1="27.3332" y1="3.3302" x2="27.3332" y2="4.445" width="0.4064" layer="1"/>
-<wire x1="27.305" y1="8.89" x2="27.3332" y2="8.8618" width="0.4064" layer="16"/>
-<wire x1="27.3332" y1="8.8618" x2="27.3332" y2="4.445" width="0.4064" layer="16"/>
+<via x="27.8412" y="4.445" extent="1-16" drill="0.35"/>
+<wire x1="25.2222" y1="1.2192" x2="27.8412" y2="3.8382" width="0.4064" layer="1"/>
+<wire x1="27.8412" y1="3.8382" x2="27.8412" y2="4.445" width="0.4064" layer="1"/>
+<wire x1="27.813" y1="8.89" x2="27.8412" y2="8.8618" width="0.4064" layer="16"/>
+<wire x1="27.8412" y1="8.8618" x2="27.8412" y2="4.445" width="0.4064" layer="16"/>
 <wire x1="21.59" y1="8.89" x2="17.78" y2="5.08" width="0.4064" layer="1"/>
 <wire x1="17.78" y1="5.08" x2="17.78" y2="2.54" width="0.4064" layer="1"/>
@@
 </signals>
 <mfgpreviewcolors>
-<mfgpreviewcolor name="soldermaskcolor" color="0xC8008000"/>
+<mfgpreviewcolor name="soldermaskcolor" color="0xC8AA00FF"/>
 <mfgpreviewcolor name="silkscreencolor" color="0xFFFEFEFE"/>
 <mfgpreviewcolor name="backgroundcolor" color="0xFF282828"/>
