File: Eagle/flying-horse-foot-v3.1.brd (EAGLE design)
At the start: 55.8 x 32.5 mm, 25 parts, among them J2 SPI6, U1 8U2-AU, Y2 16MHz

Commit message: moved from 3x2 SPI header to 6x1 SPI header
Parts:
- removed J2: SPI6, SparkFun-Connectors:2X3-NS
- added SPI6: spi_header, SparkFun-Connectors:1X06_NO_SILK
- moved U$5 5.34 mm to (5.59, 9.91)
Connections:
- removed net COL-1: J2.3, U$4.3, U1.15
- removed net COL-2: J2.4, U$4.5, U1.16
- removed net COL-3: J2.1, U$4.8, U1.17
- new net COL-1+SCLK: SPI6.5, U$4.3, U1.15
- new net COL-2+MOSI: SPI6.4, U$4.5, U1.16
- new net COL-3+MISO: SPI6.3, U$4.8, U1.17
- net D+: now also ESD.3
- net D-: now also ESD.4
- net GND: now also SPI6.1; no longer J2.6
- net RESET: now also SPI6.6; no longer J2.5
- net VCC: now also SPI6.2; no longer J2.2
Routing:
- net COL-1: track 50.4 -> 0.00 mm, vias 3 -> 0
- net COL-2: track 43.4 -> 0.00 mm, vias 2 -> 0
- net COL-3: track 43.2 -> 0.00 mm, vias 2 -> 0
- net COL-1+SCLK: track 0.00 -> 41.1 mm, vias 0 -> 2
- net COL-2+MOSI: track 0.00 -> 39.6 mm, vias 0 -> 2
- net COL-3+MISO: track 0.00 -> 39.6 mm, vias 0 -> 2
- net VCC: track 94.6 -> 85.7 mm, vias 10 -> 9
- net GND: track 89.7 -> 81.1 mm
- net RESET: track 67.9 -> 64.0 mm, vias 3 -> 2
- net ROW-13: track 18.0 -> 19.6 mm
- net ROW-14: track 21.5 -> 23.1 mm
- net ROW-16: track 30.6 -> 32.2 mm
- net ROW-15: track 23.1 -> 24.7 mm
- net D-: track 16.0 -> 17.3 mm
- net D+: track 19.4 -> 20.6 mm
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Other:
- board text added: "Adapted by: Vino Rodrigues"
- board text added: "Rev. 20210911"
- board text removed: "Rev. 20210726"
- board text removed: "SCL"

Commit message: second production run, v3.1
Parts:
- added S2: SKRKAEE020, VinoRodrigues_Custom_Eagle:SKRKAEE020
- RESET: value (none) -> 0.1 inch 2-pin
- U$1: value 74HC42D16 -> SN74HC42DR
- moved U$5 15.3 mm to (12.4, 23.6), turned to 0 degrees
- moved R2 1.55 mm to (43.6, 23.7)
- moved R1 1.52 mm to (43.6, 21.8)
- moved C5 1.37 mm to (38.6, 24.6), turned to 180 degrees
- moved R3 1.02 mm to (21.6, 28.1), turned to 0 degrees
- moved ESD 0.92 mm to (49.3, 22.6)
- moved C7 0.76 mm to (45.0, 1.91)
- moved C8 0.76 mm to (14.1, 30.7)
- moved C4 0.57 mm to (36.3, 20.7)
- moved R5 0.28 mm to (4.83, 29.2)
- moved U1 0.25 mm to (30.5, 25.5)
- moved R4 0.13 mm to (4.83, 30.9)
Connections:
- removed net COL-7: U1.21
- removed net COL-8: U1.5
- removed net COL-9: U1.26
- removed net NC: U1.8
- removed net ROW-10: U$2.1
- removed net ROW-19: U$2.11
- net GND: now also S2.1
- net RESET: now also S2.2
- net ROW-5: no longer U1.12
- net ROW-F: now also U1.12
Routing:
- net GND: track 81.1 -> 8.86 mm, vias 19 -> 13
- net VCC: track 85.7 -> 143.3 mm, vias 9 -> 8
- net ROW-5: track 41.6 -> 6.79 mm, vias 2 -> 0
- net ROW-F: track 0.00 -> 15.9 mm
- net RESET: track 64.0 -> 74.4 mm, vias 2 -> 3
- net D+: track 20.6 -> 17.0 mm
- net D-: track 17.3 -> 14.1 mm
- net HWB: track 8.13 -> 5.19 mm
- net N$1: track 10.9 -> 9.30 mm
- net ROW-A: track 58.7 -> 57.1 mm
- net ROW-B: track 57.3 -> 55.7 mm
- net N$2: track 10.5 -> 8.97 mm
- net COL-6: track 37.9 -> 36.8 mm
- net COL-12: track 40.4 -> 39.3 mm
- net ROW-17: track 42.1 -> 43.1 mm, vias 0 -> 2
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- added copper zone on layer 1, net GND
- removed copper zone on layer 1, net VCC
Other:
- board text added: "Original design by: Fredrik Atmer"
- board text removed: "Adapted by: Vino Rodrigues"

Commit message: typos
Parts:
- ISP6: value spi_header -> isp_header
- renumbered SPI6 to ISP6
Other:
- board text added: "ISP6"
- board text removed: "SPI6"
Changed lines of the file:
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@@
 <drawing>
 <settings>
-<setting alwaysvectorfont="no"/>
+<setting alwaysvectorfont="yes"/>
 <setting verticaltext="up"/>
 </settings>
@@
 <text x="45.1485" y="16.764" size="0.6096" layer="21" font="vector" rot="R270" align="bottom-center">RESET</text>
 <text x="26.035" y="25.4" size="0.6096" layer="21" font="vector" rot="R45" align="center-left">ATMEGA32U2</text>
-<text x="12.7" y="28.575" size="0.6096" layer="21" font="vector" rot="R270" align="center-left">74HC42</text>
-<text x="46.355" y="3.81" size="0.6096" layer="21" font="vector" rot="R90" align="center-left">74HC42</text>
+<text x="13.462" y="27.305" size="0.6096" layer="21" font="vector" rot="R270" align="center-left">74HC42</text>
+<text x="46.101" y="4.826" size="0.6096" layer="21" font="vector" rot="R90" align="center-left">74HC42</text>
 <text x="39.37" y="7.62" size="0.6096" layer="21" font="vector" rot="R90" align="center-left">MK6-5-B</text>
 <text x="3.683" y="1.27" size="0.8128" layer="26" rot="MR270" align="bottom-right">github.com/Tecsmith/flying-horse-foot</text>
@@
 <text x="9.906" y="9.652" size="0.6096" layer="25" rot="R90" align="top-center">MOSI</text>
 <text x="9.906" y="4.572" size="0.6096" layer="25" rot="R90" align="top-center">VCC</text>
-<text x="6.858" y="2.032" size="0.8128" layer="26" ratio="16" rot="MR90" align="top-center">SPI6</text>
+<text x="6.858" y="2.032" size="0.8128" layer="26" ratio="16" rot="MR90" align="top-center">ISP6</text>
 <rectangle x1="41.6433" y1="17.6149" x2="41.8973" y2="17.6403" layer="26"/>
 <rectangle x1="41.6179" y1="17.6403" x2="41.9481" y2="17.6657" layer="26"/>
@@
 <text x="7.112" y="14.986" size="0.6096" layer="26" rot="MR90" align="top-center">RESET</text>
 <text x="4.572" y="8.001" size="0.6096" layer="25" rot="R180" align="top-center">RESET</text>
+<circle x="34.0995" y="25.527" radius="0.567959375" width="0.1524" layer="21"/>
 </plain>
 <attributes>
@@
 </element>
 <element name="U$5" library="VinoRodrigues_Custom_Eagle" package="TECSMITH-LOGO" value="TECSMITH-LOGO" x="12.446" y="23.622" smashed="yes" rot="MR0"/>
-<element name="SPI6" library="SparkFun-Connectors" package="1X06_NO_SILK" value="spi_header" x="8.382" y="2.032" smashed="yes" rot="R90">
+<element name="ISP6" library="SparkFun-Connectors" package="1X06_NO_SILK" value="isp_header" x="8.382" y="2.032" smashed="yes" rot="R90">
 <attribute name="NAME" x="8.382" y="16.383" size="0.6096" layer="25" font="vector" ratio="20" align="bottom-center"/>
 <attribute name="VALUE" x="10.414" y="0.762" size="0.6096" layer="27" font="vector" ratio="20" rot="R90"/>
@@
 <wire x1="10.16" y1="17.526" x2="10.1445" y2="17.5105" width="0.3048" layer="16"/>
 <contactref element="ESD" pad="2"/>
-<contactref element="SPI6" pad="1"/>
+<contactref element="ISP6" pad="1"/>
 <via x="13.335" y="22.7965" extent="1-16" drill="0.35"/>
 <via x="18.161" y="23.8125" extent="1-16" drill="0.35"/>
@@
 <wire x1="5.842" y1="18.669" x2="5.842" y2="19.939" width="0.3048" layer="1"/>
 <via x="5.842" y="19.939" extent="1-16" drill="0.35"/>
-<contactref element="SPI6" pad="4"/>
+<contactref element="ISP6" pad="4"/>
 <wire x1="6.0961875" y1="11.9378125" x2="8.382" y2="9.652" width="0.3048" layer="1"/>
 <wire x1="5.842" y1="19.939" x2="2.525" y2="23.256" width="0.3048" layer="16"/>
@@
 <wire x1="4.572" y1="17.78" x2="4.048" y2="17.256" width="0.3048" layer="16"/>
 <wire x1="4.048" y1="17.256" x2="1.4003" y2="17.256" width="0.3048" layer="16"/>
-<contactref element="SPI6" pad="3"/>
+<contactref element="ISP6" pad="3"/>
 <wire x1="5.334" y1="10.16" x2="8.382" y2="7.112" width="0.3048" layer="1"/>
 <wire x1="5.334" y1="17.78" x2="5.334" y2="10.16" width="0.3048" layer="1"/>
@@
 <wire x1="5.842" y1="21.209" x2="5.842" y2="21.1455" width="0.3048" layer="1"/>
 <wire x1="5.842" y1="21.1455" x2="6.731" y2="20.2565" width="0.3048" layer="1"/>
-<contactref element="SPI6" pad="5"/>
+<contactref element="ISP6" pad="5"/>
 <wire x1="6.731" y1="13.843" x2="8.382" y2="12.192" width="0.3048" layer="1"/>
 <wire x1="6.731" y1="20.2565" x2="6.731" y2="13.843" width="0.3048" layer="1"/>
@@
 <wire x1="34.544" y1="29.718" x2="37.846" y2="26.416" width="0.4064" layer="16"/>
 <contactref element="ESD" pad="5"/>
-<contactref element="SPI6" pad="2"/>
+<contactref element="ISP6" pad="2"/>
 <via x="5.842" y="23.622" extent="1-16" drill="0.35"/>
 <via x="3.302" y="27.686" extent="1-16" drill="0.35"/>
@@
 <wire x1="40.6273" y1="18.5547" x2="41.148" y2="18.034" width="0.3048" layer="16"/>
 <wire x1="41.148" y1="18.034" x2="43.561" y2="18.034" width="0.3048" layer="16"/>
-<contactref element="SPI6" pad="6"/>
+<contactref element="ISP6" pad="6"/>
 <wire x1="5.81695625" y1="22.39045625" x2="7.366" y2="20.8414125" width="0.3048" layer="1"/>
 <wire x1="7.366" y1="20.8414125" x2="7.366" y2="15.748" width="0.3048" layer="1"/>
@@
 </signals>
 <mfgpreviewcolors>
-<mfgpreviewcolor name="soldermaskcolor" color="0xC8008000"/>
-<mfgpreviewcolor name="silkscreencolor" color="0xFFFEFEFE"/>
+<mfgpreviewcolor name="soldermaskcolor" color="0xC8AA55FF"/>
+<mfgpreviewcolor name="silkscreencolor" color="0xFFFFFFFF"/>
 <mfgpreviewcolor name="backgroundcolor" color="0xFF282828"/>
 <mfgpreviewcolor name="coppercolor" color="0xFFFFBF00"/>

Commit message: caps and scr led swap
Connections:
- removed net LED-SCROLL: R5.1, U$4.2
- new net LED-SCR: R4.1, U$4.1
- net LED-CAPS: now also R5.1, U$4.2; no longer R4.1, U$4.1
Routing:
- net LED-SCR: track 0.00 -> 2.75 mm
- net LED-SCROLL: track 2.59 -> 0.00 mm
Changed lines of the file:
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@@
 <drawing>
 <settings>
-<setting alwaysvectorfont="yes"/>
+<setting alwaysvectorfont="no"/>
 <setting verticaltext="up"/>
 </settings>
@@
 <wire x1="49.53" y1="18.034" x2="36.83" y2="30.734" width="0.3048" layer="16"/>
 </signal>
-<signal name="LED-CAPS">
+<signal name="LED-SCR">
 <contactref element="U$4" pad="1"/>
 <contactref element="R4" pad="1"/>
@@
 <wire x1="1.4003" y1="31.256" x2="1.4003" y2="31.2387" width="0.3048" layer="1"/>
 </signal>
-<signal name="LED-SCROLL">
+<signal name="LED-CAPS">
 <contactref element="U$4" pad="2"/>
 <contactref element="R5" pad="1"/>

Commit message: ·
Parts:
- S2: device VinoRodrigues_Custom_Eagle:SKRKAEE020 -> SilvinoR_Custom_Eagle:SKRKAEE020
- U$5: device VinoRodrigues_Custom_Eagle:TECSMITH-LOGO -> SilvinoR_Custom_Eagle:TECSMITH-LOGO
Other:
- board text added: "2021 adaptation by Silvino Rodrigues"
- board text removed: "2021 adaptation by Vino Rodrigues"
Changed lines of the file:
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@@
 <rectangle x1="7.112" y1="0.762" x2="9.652" y2="3.302" layer="22"/>
 <text x="9.7282" y="20.9042" size="0.8128" layer="26" rot="MR270" align="bottom-center">2021 adaptation by
-Vino Rodrigues</text>
+Silvino Rodrigues</text>
 <wire x1="40.132" y1="19.304" x2="40.386" y2="19.05" width="0.1524" layer="22"/>
 <wire x1="40.386" y1="19.05" x2="40.386" y2="17.018" width="0.1524" layer="22"/>
@@
 <attribute name="SUPPLIER" value="TEXAS INSTRUMENTS" x="49.276" y="22.606" size="1.778" layer="27" rot="R90" display="off"/>
 </element>
-<element name="U$5" library="VinoRodrigues_Custom_Eagle" package="TECSMITH-LOGO" value="TECSMITH-LOGO" x="12.446" y="23.622" smashed="yes" rot="MR0"/>
+<element name="U$5" library="SilvinoR_Custom_Eagle" package="TECSMITH-LOGO" value="TECSMITH-LOGO" x="12.446" y="23.622" smashed="yes" rot="MR0"/>
 <element name="ISP6" library="SparkFun-Connectors" package="1X06_NO_SILK" value="isp_header" x="8.382" y="2.032" smashed="yes" rot="R90">
 <attribute name="NAME" x="8.382" y="16.383" size="0.6096" layer="25" font="vector" ratio="20" align="bottom-center"/>
 <attribute name="VALUE" x="10.414" y="0.762" size="0.6096" layer="27" font="vector" ratio="20" rot="R90"/>
 </element>
-<element name="S2" library="VinoRodrigues_Custom_Eagle" package="SKRKAEE020" value="SKRKAEE020" x="4.572" y="5.08" smashed="yes" rot="R90">
+<element name="S2" library="SilvinoR_Custom_Eagle" package="SKRKAEE020" value="SKRKAEE020" x="4.572" y="5.08" smashed="yes" rot="R90">
 <attribute name="VALUE" x="9.382" y="1.7" size="1.778" layer="27" rot="R90"/>
 </element>
